File: hardware/nyx2/nyx2.kicad_pcb (KiCad board)
At the start: 4 copper layers, 51 x 21 mm, 48 parts, among them J5 USB4215-03-A, U1 RP2350, U2 ESP-PSRAM32, U3 W25Q128JVS, U4 NCP1117 3.3, Y1 ASE-12MHz

Commit message: Nyx 2B released + repo cleanup
Routing:
- net VBUS: track 72.3 -> 73.8 mm
- net /D+: track 28.6 -> 27.5 mm
